Commit message: changed cylinder into box

File: first.urdf (robot description, URDF)
Before this commit: robot firsttry, 2 links, 1 joints
Links:
- link base_link: geometry visual box size=0.6 0.2 0.3

Commit message: proper robot urdf file (checked)

File: first.urdf (robot description, URDF)
Before this commit: robot firsttry, 2 links, 1 joints
Links:
- link sonar0: geometry visual box size=0.05 0.05 0.05
Joints:
- joint sonar0_joint: axis 0 0 1 -> (none)
