Commit message: sonar name changed

File: robotURDF.urdf (robot description, URDF)
Before this commit: robot IMRrobot, 7 links, 6 joints
Joints:
- joint sonar0_joint: origin xyz=0.2425 0 0.15 rpy=0 0 0 -> xyz=0.135 0.1875 0.15 rpy=0 0 1.57075
- joint sonar2_joint: origin xyz=0.225 -0.125 0.15 rpy=0 0 -0.785398 -> xyz=0.2425 0 0.15 rpy=0 0 0
- joint sonar3_joint: origin xyz=0.135 -0.1875 0.15 rpy=0 0 -1.57075 -> xyz=0.225 -0.125 0.15 rpy=0 0 -0.785398
- joint sonar4_joint: origin xyz=0.135 0.1875 0.15 rpy=0 0 1.57075 -> xyz=0.135 -0.1875 0.15 rpy=0 0 -1.57075
