Commit message: meshes added

File: urdf/robotURDF.urdf.xacro (robot description, xacro)
@@ -1,4 +1,4 @@
 <?xml version="1.0"?>
-<robot name="IMRrobot">
+<robot name="IMRrobot" xmlns:xacro="http://ros.org/wiki/xacro">
    <material name="white">
       <color rgba="1 1 1 1"/>
@@ -16,4 +16,10 @@
   </link>
   <!-- LIDAR -->
+  <joint name="lidar_link_joint" type="fixed">
+    <axis xyz="1 0 0"/>
+    <parent link="base_link"/>
+    <child link="lidar_link"/>.
+    <origin rpy="0 0 0" xyz="0.125 0 0.25"/>
+  </joint>
   <link name="lidar_link">
     <visual>
@@ -25,11 +31,12 @@
     </visual>
   </link>
-  <joint name="lidar_link_joint" type="fixed">
-    <axis xyz="1 0 0"/>
+   <!-- SONAR0 -->
+  <joint name="sonar0_joint" type="fixed">
     <parent link="base_link"/>
-    <child link="lidar_link"/>.
-    <origin rpy="0 0 0" xyz="0.125 0 0.25"/>
+    <child link="sonar0"/>
+    <origin rpy="0 0 1.57075" xyz="0.135 0.1875 0.15"/>
+   <!-- <axis xyz="0 0 1"/>
+    <origin xyz="0 -0.22 0.25"/> -->
   </joint>
-   <!-- SONAR0 -->
   <link name="sonar0">
     <visual>
@@ -42,12 +49,12 @@
     </visual>
   </link>
-  <joint name="sonar0_joint" type="fixed">
+<!-- SONAR1 -->
+  <joint name="sonar1_joint" type="fixed">
     <parent link="base_link"/>
-    <child link="sonar0"/>
-    <origin rpy="0 0 1.57075" xyz="0.135 0.1875 0.15"/>
+    <child link="sonar1"/>
+    <origin rpy="0 0 0.785398" xyz="0.225 0.125 0.15"/>
    <!-- <axis xyz="0 0 1"/>
     <origin xyz="0 -0.22 0.25"/> -->
   </joint>
-<!-- SONAR1 -->
   <link name="sonar1">
     <visual>
@@ -60,12 +67,12 @@
     </visual>
   </link>
-  <joint name="sonar1_joint" type="fixed">
+ <!-- SONAR2 -->
+  <joint name="sonar2_joint" type="fixed">
     <parent link="base_link"/>
-    <child link="sonar1"/>
-    <origin rpy="0 0 0.785398" xyz="0.225 0.125 0.15"/>
+    <child link="sonar2"/>
+    <origin rpy="0 0 0" xyz="0.2425 0 0.15"/>
    <!-- <axis xyz="0 0 1"/>
     <origin xyz="0 -0.22 0.25"/> -->
   </joint>
- <!-- SONAR2 -->
   <link name="sonar2">
     <visual>
@@ -78,12 +85,12 @@
     </visual>
   </link>
-  <joint name="sonar2_joint" type="fixed">
+ <!-- SONAR3 -->
+  <joint name="sonar3_joint" type="fixed">
     <parent link="base_link"/>
-    <child link="sonar2"/>
-    <origin rpy="0 0 0" xyz="0.2425 0 0.15"/>
+    <child link="sonar3"/>
+    <origin rpy="0 0 -0.785398" xyz="0.225 -0.125 0.15"/>
    <!-- <axis xyz="0 0 1"/>
     <origin xyz="0 -0.22 0.25"/> -->
   </joint>
- <!-- SONAR3 -->
   <link name="sonar3">
     <visual>
@@ -96,12 +103,12 @@
     </visual>
   </link>
-  <joint name="sonar3_joint" type="fixed">
+   <!-- SONAR4 -->
+  <joint name="sonar4_joint" type="fixed">
     <parent link="base_link"/>
-    <child link="sonar3"/>
-    <origin rpy="0 0 -0.785398" xyz="0.225 -0.125 0.15"/>
+    <child link="sonar4"/>
+    <origin rpy="0 0 -1.57075" xyz="0.135 -0.1875 0.15"/>
    <!-- <axis xyz="0 0 1"/>
     <origin xyz="0 -0.22 0.25"/> -->
   </joint>
-   <!-- SONAR4 -->
   <link name="sonar4">
     <visual>
@@ -114,10 +121,3 @@
     </visual>
   </link>
-  <joint name="sonar4_joint" type="fixed">
-    <parent link="base_link"/>
-    <child link="sonar4"/>
-    <origin rpy="0 0 -1.57075" xyz="0.135 -0.1875 0.15"/>
-   <!-- <axis xyz="0 0 1"/>
-    <origin xyz="0 -0.22 0.25"/> -->
-  </joint>
 </robot>
