Commit message: Tested with HW, rotation issue

File: urdf/robotURDF-2.urdf (robot description, URDF)
Before this commit: robot IMRrobot, 9 links, 8 joints
Joints:
- joint imu_link_joint: axis 1 0 0 -> (none); origin xyz=0 0 0 rpy=0 0 0 -> (none); parent sensor_head_link -> base_link
- joint sensor_head_link_joint: origin xyz=0 0 0.25 rpy=0 0 0 -> xyz=0 0 0 rpy=0 0 0; parent base_link -> imu_link

Commit message: rotation issue resolved

File: urdf/robotURDF-2.urdf (robot description, URDF)
Before this commit: robot IMRrobot, 9 links, 8 joints
Joints:
- joint sensor_head_link_joint: origin xyz=0 0 0 rpy=0 0 0 -> xyz=0 0 0 rpy=3.14159 0 0
